File: LED_DRV.kicad_sch (KiCad schematic)
At the start: 16 parts, among them U1 LGS63042EP

Commit message: Add panel project.
Parts:
- removed C2: 4.7uF, 001_GN_RCL_SMD:C0805(2012M), symbol 001_Basic_PassiveComponents:101_Capacitor
- added D10, D11, D7, D8, D9: BXEN-65E-13H, 002_GN_TWO-PIN_PLASTIC_SMD:LED2835M, symbol 002_Basic_SingleSemiconductor:008_Diode_LightEmitting
- added P1, P2, P3, P4, P5, P6: Pad_Square, 302_MECH_PAD:SMP-Q_2020, symbol 301_Link_Pad:Pad_Square
- D2, D3, D4, D5, D6: footprint 002_GN_TWO-PIN_PLASTIC_SMD:LED0603(1608M) -> 002_GN_TWO-PIN_PLASTIC_SMD:LED2835M
- L1: footprint 008_GN_POWER-CHOKE_SMD:MC-0530 -> 008_GN_POWER-CHOKE_SMD:MC-2520
- R2: footprint 001_GN_RCL_SMD:R0603(1608M) -> 001_GN_RCL_SMD:R0805(2012M)
Connections:
- net DIM: now also P3.PAD, P6.PAD
- net GND: now also U1.EP, D11.1 (Cathode), P2.PAD, P5.PAD
- net LED_A: now also D7.2 (Anode)
- net VBUS: now also P1.PAD, P4.PAD
- new net: D7.1 (Cathode), D8.2 (Anode)
- new net: D8.1 (Cathode), D9.2 (Anode)
- new net: D10.2 (Anode), D9.1 (Cathode)
- new net: D10.1 (Cathode), D11.2 (Anode)
Other:
- moved on the sheet: C1, C3, C4, D1, L1, R1, R2, R3, R4

Commit message: Daily update
Parts:
- C1: value 4.7uF -> 22uF
- L1: value 10uH -> 22uH
- R1: value 2R -> 1R
Changed lines of the file:
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@@
       (effects (font (size 1.27 1.27)) (justify left))
     )
-    (property "Value" "4.7uF" (at 76.2 77.47 90)
+    (property "Value" "22uF" (at 76.2 77.47 90)
       (effects (font (size 1.27 1.27)) (justify left))
     )
@@
       (effects (font (size 1.27 1.27)))
     )
-    (property "Value" "10uH" (at 81.28 58.42 0)
+    (property "Value" "22uH" (at 81.28 58.42 0)
       (effects (font (size 1.27 1.27)))
     )
@@
       (effects (font (size 1.27 1.27)))
     )
-    (property "Value" "2R" (at 124.46 73.66 0)
-      (effects (font (size 1.27 1.27)))
-    )
+    (property "Value" "1R" (at 124.46 73.66 0)
+      (effects (font (size 1.27 1.27)))
+    )
