File: LED_CTRL/LED_CTRL.kicad_pcb (KiCad board)
At the start: 2 copper layers, 31.2 x 17.5 mm, 5 parts, among them P1 EN+, P2 EN-, P3 END, P4 MID, P5 STR

Commit message: Update before RUN
Parts:
- added C1: 100nF, 001_GN_RCL_SMD:C0402(1005M), F.Cu at (75.5, 99.9)
- added C10: 22uF, 001_GN_RCL_SMD:C0603(1608M), F.Cu at (79.4, 100.6)
- added C2: 100nF, 001_GN_RCL_SMD:C0402(1005M), F.Cu at (73.9, 99.9)
- added C3: 1uF, 001_GN_RCL_SMD:C0402(1005M), F.Cu at (77.0, 104.2)
- added C4: 1uF, 001_GN_RCL_SMD:C0402(1005M), F.Cu at (74.1, 105.9)
- added C5: 100nF, 001_GN_RCL_SMD:C0402(1005M), F.Cu at (84.9, 105.2)
- added C6: 330pF, 001_GN_RCL_SMD:C0402(1005M), F.Cu at (78.2, 103.9)
- added C8: 22uF, 001_GN_RCL_SMD:C0603(1608M), F.Cu at (84.1, 97.9)
- added C9: 1uF, 001_GN_RCL_SMD:C0402(1005M), F.Cu at (84.2, 99.9)
- added D1: 1N5819, 002_GN_TWO-PIN_PLASTIC_SMD:SOD-323, F.Cu at (87.1, 105.4)
- added D2: 1N5819, 002_GN_TWO-PIN_PLASTIC_SMD:SOD-323, F.Cu at (87.1, 103.6)
- added D3: LMBR240ET1G, 002_GN_TWO-PIN_PLASTIC_SMD:SOD-323HE, F.Cu at (79.4, 98.0)
- added L1: 22uH, 008_GN_POWER-CHOKE_SMD:MC-2520, F.Cu at (81.9, 97.6)
- added P10: P-, 302_MECH_PAD:SMP-Q_2020, F.Cu at (73.8, 108.5)
- added P11: PWM, 302_MECH_PAD:SMP-Q_2020, F.Cu at (87.5, 108.5)
- added P12: VLED, 302_MECH_PAD:SMP-Q_2020, F.Cu at (83.8, 108.5)
- added P13: GND, 302_MECH_PAD:SMP-Q_2020, F.Cu at (91.2, 108.5)
- added P6: CELL2, 302_MECH_PAD:SMP-Q_2020, F.Cu at (87.5, 94.0)
- added P7: CELL1, 302_MECH_PAD:SMP-Q_2020, F.Cu at (83.8, 94.0)
- added P8: CELL-, 302_MECH_PAD:SMP-Q_2020, F.Cu at (80.0, 94.0)
- added P9: P+, 302_MECH_PAD:SMP-Q_2020, F.Cu at (77.5, 108.5)
- added Q1: MDD2300, 003_GN_SMALL-SEMI_SMD:SOT-23, F.Cu at (76.5, 94.5)
- added Q2: MDD2300, 003_GN_SMALL-SEMI_SMD:SOT-23, F.Cu at (73.1, 94.5)
- added Q3: MDD2301, 003_GN_SMALL-SEMI_SMD:SOT-23, F.Cu at (86.5, 98.0)
- added Q4: MDD2300, 003_GN_SMALL-SEMI_SMD:SOT-23, F.Cu at (87.0, 101.1)
- added R1: 330R, 001_GN_RCL_SMD:R0402(1005M), F.Cu at (75.5, 100.9)
- added R2: 330R, 001_GN_RCL_SMD:R0402(1005M), F.Cu at (73.9, 100.9)
- added R3: 2k, 001_GN_RCL_SMD:R0402(1005M), F.Cu at (72.5, 100.4)
- added R4: 330R, 001_GN_RCL_SMD:R0402(1005M), F.Cu at (84.5, 101.2)
- added R5: 330R, 001_GN_RCL_SMD:R0402(1005M), F.Cu at (84.9, 103.5)
- added R6: 100k, 001_GN_RCL_SMD:R0402(1005M), F.Cu at (88.5, 98.0)
- added R7: 220k, 001_GN_RCL_SMD:R0402(1005M), F.Cu at (77.9, 100.2)
- added R8: 10k, 001_GN_RCL_SMD:R0402(1005M), F.Cu at (77.9, 101.2)
- added U1: LM555CMM, 004_GN_MIDDLE-SEMI_SMD:MSOP-8_3030, F.Cu at (81.5, 104.5)
- added U2: ME6215C33M5G, 003_GN_SMALL-SEMI_SMD:SOT-23-5, F.Cu at (74.8, 103.8)
- added U3: ME4212BM6G, 003_GN_SMALL-SEMI_SMD:SOT-23-6, F.Cu at (74.5, 97.8)
- added U4: HX3608, 003_GN_SMALL-SEMI_SMD:SOT-23-6, F.Cu at (81.9, 100.6)
Connections:
- P1 pad PAD: unconnected-(P1-PadPAD) -> +7.5V
- P2 pad PAD: unconnected-(P2-PadPAD) -> Net-(P2-PadPAD)
- P3 pad PAD: unconnected-(P3-PadPAD) -> Net-(D2-Anode)
- P4 pad PAD: unconnected-(P4-PadPAD) -> /MID
- P5 pad PAD: unconnected-(P5-PadPAD) -> Net-(D1-Cathode)
Routing:
- net Net-(P2-PadPAD): track 0.00 -> 21.4 mm
- net /MID: track 0.00 -> 18.3 mm, vias 0 -> 2
- net Net-(P7-PadPAD): track 0.00 -> 15.9 mm, vias 0 -> 2
- net +5V: track 0.00 -> 13.3 mm, vias 0 -> 2
- net /EN: track 0.00 -> 11.1 mm
- net /PWM: track 0.00 -> 9.82 mm, vias 0 -> 5
- net Net-(D1-Cathode): track 0.00 -> 7.48 mm
- net GND: track 0.00 -> 7.02 mm, vias 0 -> 45
- net Net-(Q1-Source): track 0.00 -> 6.57 mm
- net Net-(U4-FB): track 0.00 -> 4.78 mm
- net Net-(D2-Anode): track 0.00 -> 4.73 mm
- net Net-(Q3-Gate): track 0.00 -> 4.56 mm
- net Net-(Q3-Drain): track 0.00 -> 4.17 mm
- net /DSG: track 0.00 -> 4.10 mm
- net Net-(U3-Vin): track 0.00 -> 3.78 mm
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- added copper zone on B.Cu, net +7.5V
- added copper zone on F.Cu, net +7.5V
- added copper zone on B.Cu, net /PWM
- added copper zone on B.Cu, net GND
- added copper zone on F.Cu, net GND
- added copper zone on F.Cu, net Net-(D3-Anode)
- added copper zone on F.Cu, net Net-(Q1-Drain)
- added copper zone on F.Cu, net Net-(Q1-Source)
- added copper zone on F.Cu, net Net-(Q3-Drain)
- added copper zone on B.Cu, net VDC
- added copper zone on F.Cu, net VDC
Other:
- board text added: "LED_CTRL_v1.0(240516)"
