File: LED_CTRL/LED_CTRL.kicad_sch (KiCad schematic)
At the start: 5 parts, among them P1 EN+, P2 EN-, P3 END, P4 MID, P5 STR

Commit message: Update before RUN
Parts:
- added C1, C2, C5: 100nF, 001_GN_RCL_SMD:C0402(1005M), symbol 001_Basic_PassiveComponents:101_Capacitor
- added C10, C8: 22uF, 001_GN_RCL_SMD:C0603(1608M), symbol 001_Basic_PassiveComponents:101_Capacitor
- added C3, C4, C9: 1uF, 001_GN_RCL_SMD:C0402(1005M), symbol 001_Basic_PassiveComponents:101_Capacitor
- added C6: 330pF, 001_GN_RCL_SMD:C0402(1005M), symbol 001_Basic_PassiveComponents:101_Capacitor
- added D1, D2: 1N5819, 002_GN_TWO-PIN_PLASTIC_SMD:SOD-323, symbol 002_Basic_SingleSemiconductor:002_Diode_Schottky
- added D3: LMBR240ET1G, 002_GN_TWO-PIN_PLASTIC_SMD:SOD-323HE, symbol 002_Basic_SingleSemiconductor:002_Diode_Schottky
- added L1: 22uH, 008_GN_POWER-CHOKE_SMD:MC-2520, symbol 001_Basic_PassiveComponents:202_PowerChoke
- added P10: P-, 302_MECH_PAD:SMP-Q_2020, symbol 301_Link_Pad:Pad_Square
- added P11: PWM, 302_MECH_PAD:SMP-Q_2020, symbol 301_Link_Pad:Pad_Square
- added P12: VLED, 302_MECH_PAD:SMP-Q_2020, symbol 301_Link_Pad:Pad_Square
- added P13: GND, 302_MECH_PAD:SMP-Q_2020, symbol 301_Link_Pad:Pad_Square
- added P6: CELL2, 302_MECH_PAD:SMP-Q_2020, symbol 301_Link_Pad:Pad_Square
- added P7: CELL1, 302_MECH_PAD:SMP-Q_2020, symbol 301_Link_Pad:Pad_Square
- added P8: CELL-, 302_MECH_PAD:SMP-Q_2020, symbol 301_Link_Pad:Pad_Square
- added P9: P+, 302_MECH_PAD:SMP-Q_2020, symbol 301_Link_Pad:Pad_Square
- added Q1, Q2, Q4: MDD2300, 003_GN_SMALL-SEMI_SMD:SOT-23, symbol 002_Basic_SingleSemiconductor:201_MOSFET_N-ch
- added Q3: MDD2301, 003_GN_SMALL-SEMI_SMD:SOT-23, symbol 002_Basic_SingleSemiconductor:202_MOSFET_P-ch
- added R1, R2, R4, R5: 330R, 001_GN_RCL_SMD:R0402(1005M), symbol 001_Basic_PassiveComponents:001_Resistor
- added R3: 2k, 001_GN_RCL_SMD:R0402(1005M), symbol 001_Basic_PassiveComponents:001_Resistor
- added R6: 100k, 001_GN_RCL_SMD:R0402(1005M), symbol 001_Basic_PassiveComponents:001_Resistor
- added R7: 220k, 001_GN_RCL_SMD:R0402(1005M), symbol 001_Basic_PassiveComponents:001_Resistor
- added R8: 10k, 001_GN_RCL_SMD:R0402(1005M), symbol 001_Basic_PassiveComponents:001_Resistor
- added U1: LM555CMM, 004_GN_MIDDLE-SEMI_SMD:MSOP-8_3030, symbol 102_IntegratedCircuit_Logic:NE555
- added U2: CJ6376B33M, 003_GN_SMALL-SEMI_SMD:SOT-23-5, symbol 203_Power_LDO:ME6215C33M5G
- added U3: ME4212BM6G, 003_GN_SMALL-SEMI_SMD:SOT-23-6, symbol LED_CTRL:ME4212BM6G
- added U4: HX3608, 003_GN_SMALL-SEMI_SMD:SOT-23-6, symbol 204_Power_SMPS-Convertor:HX3608
Connections:
- net MID: now reaches P4.PAD
- net MID: now also C6.1, U1.2 (TRIG), U1.6 (THRS)
- net at P2.PAD: now also R4.1
- net at P3.PAD: now also D2.2 (Anode)
- net +7.5V: now reaches P1.PAD
- net +7.5V: now also C3.1, P6.PAD, P9.PAD, Q3.2 (Source), R1.1, R6.1, U2.1 (Vin)
- net at P5.PAD: now also D1.1 (Cathode)
- new net: C2.2, P8.PAD, Q1.2 (Source), U3.6 (GND)
- new net: C8.1, C9.1, L1.1, Q3.3 (Drain), U4.5 (VIN)
- new net: R3.1, U3.3 (CS)
- new net: R7.1, R8.2, U4.3 (FB)
- new net: Q3.1 (Gate), Q4.2 (Source), R6.2
- new net: P7.PAD, R2.1
- new net: C1.2, C2.1, R2.2, U3.4 (Vmid)
- new net: C5.1, U1.5 (VREG)
- new net: D3.2 (Anode), L1.2, U4.1 (SW)
- new net: Q2.1 (Gate), U3.2 (OC)
- new net: Q1.3 (Drain), Q2.3 (Drain)
- new net: Q1.1 (Gate), U3.1 (OD)
- new net: C1.1, R1.2, U3.5 (Vin)
- new net +5V: C4.1, R5.1, U1.4 (RST), U1.8 (Vin), U2.5 (Vout)
- new net DSG: D1.2 (Anode), D2.1 (Cathode), R5.2, U1.7 (DCHG)
- new net EN: Q4.1 (Gate), R4.2, U2.3 (EN), U4.4 (EN)
- new net GND: C10.2, C3.2, C4.2, C5.2, C6.2, C8.2, C9.2, P10.PAD, P13.PAD, Q2.2 (Source), Q4.3 (Drain), R3.2, R8.1, U1.1 (GND), U2.2 (GND), U4.2 (GND), U4.6 (NC)
- new net PWM: P11.PAD, U1.3 (OUT)
- new net VDC: C10.1, D3.1 (Cathode), P12.PAD, R7.2
Other:
- moved on the sheet: P1, P2, P3, P4, P5
